Commit message: 24 marzo

File: urdf/jetracer.xacro (robot description, xacro)
@@ -4,9 +4,96 @@
     <color rgba="0 0 0 1"/>
   </material>
+  <material name="blue">
+    <color rgba="0.5 0.5 0.5 1"/>
+  </material>
+  <joint name="camera_joint" type="fixed">
+      <origin xyz="0.17 0 0.1" rpy="0 0 0" />
+      <parent link="base"/>
+      <child link="camera" />
+      <axis xyz="0 1 0"/>
+  </joint>
+  <!-- CAMARA -->
+  <link name="camera">
+    <inertial>
+      <mass value="0.1"/>
+      <origin xyz="0 0 0" rpy="0 0 0"/>
+      <inertia
+        ixx="1e-6" ixy="0.0" ixz="0.0"
+        iyy="1e-6" iyz="0.0"
+        izz="1e-6"
+      />
+    </inertial>
+    <collision>
+      <origin xyz="0 0 0" rpy="0 0 0"/>
+      <geometry>
+        <box size="0.05 0.05 0.05"/>
+      </geometry>
+    </collision>
+    <visual>
+      <origin xyz="0 0 0" rpy="0 0 0"/>
+      <geometry>
+        <box size="0.05 0.05 0.05"/>
+      </geometry>
+      <material name="blue"/>
+    </visual>
+  </link>
+  <!--LASER-->
+    <joint name="hokuyo_joint" type="fixed">
+      <origin xyz="0.10 -0.03 0.15" rpy="0 0 0" />
+      <parent link="base"/>
+      <child link="hokuyo" />
+      <axis xyz="0 1 0"/>
+    </joint>
+  <link name="hokuyo">
+    <inertial>
+      <mass value="1e-5"/>
+      <origin xyz="0 0 0" rpy="0 0 0"/>
+      <inertia
+        ixx="1e-6" ixy="0.0" ixz="0.0"
+        iyy="1e-6" iyz="0.0"
+        izz="1e-6"
+      />
+    </inertial>
+    <collision>
+      <origin xyz="0 0 0" rpy="0 0 0"/>
+      <geometry>
+        <box size="0.1 0.1 0.1"/>
+      </geometry>
+    </collision>
+    <visual>
+      <origin xyz="0 0 0" rpy="0 0 0"/>
+      <geometry>
+        <mesh filename="package://trixy/meshes/hokuyo.dae"/>
+      </geometry>
+    </visual>
+  </link>
+    <link name="robot_footprint"></link>
+    <joint name="robot_footprint_joint" type="fixed">
+      <origin xyz="0 0 0" rpy="0 0 0" />
+      <parent link="robot_footprint"/>
+      <child link="base" />
+    </joint>
+<!--BASE-->
   <link name="base">
-    <visual>
-      <orgin rpy="0 0 0" xyz="0 0 0"/>
-      <geometry>
-        <box size="1 2 0.3"/>
+    <pose>0 0 0 0 0 0</pose>
+    <inertial>
+      <mass value="25.0"/>
+      <origin xyz="0 0 0.05" rpy=" 0 0 0"/>
+      <inertia
+          ixx="0.1" ixy="0" ixz="0"
+          iyy="0.1" iyz="0"
+          izz="0.1"
+      />
+    </inertial>
+    <collision name='base_collision'>
+      <origin xyz="0 0 0.05" rpy=" 0 0 0"/>
+      <geometry>
+        <box size="0.6 0.3 0.05"/>
+      </geometry>
+    </collision>
+    <visual name='base_visual'>
+      <origin xyz="0 0 0.05" rpy=" 0 0 0"/>
+      <geometry>
+        <box size="0.6 0.3 0.05"/>
       </geometry>
     </visual>
@@ -16,27 +103,57 @@
     <axis xyz="0 0 1"/>
     <limit effort="1000.0" lower="-0.4" upper="0.4" velocity="0.5"/>
-    <origin rpy="0 0 0" xyz="-0.5 0.8 0"/>
+    <origin rpy="0 0 0" xyz="0.2 0.25 0"/>
     <parent link="base"/>
     <child link="fl_wheel_link"/>
   </joint>
   <link name="fl_wheel_link">
-    <visual>
-      <orgin rpy="0 0 0" xyz="-0.7 0.8 0"/>
+    <inertial>
+      <mass value="1e-4"/>
+      <origin rpy="0 0 0" xyz="0.7 0.8 0"/>
+      <inertia
+        ixx="0.1" ixy="0.0" ixz="0.0"
+        iyy="0.1" iyz="0.0"
+        izz="0.1"
+      />
+    </inertial>
+    <collision>
+     <origin rpy="0 0 0" xyz="0.7 0.8 0"/>
       <geometry>
         <box size="0 0 0"/>
       </geometry>
+    </collision>
+    <visual>
+      <origin rpy="0 0 0" xyz="0.7 0.8 0"/>
+     <geometry>
+        <box size="0 0 0"/>
+      </geometry>
     </visual>
   </link>
   <joint name="fl_wheel_joint" type="continuous">
-    <axis xyz="0 0 1"/>
-    <origin rpy="0 1.57 0" xyz="-0.2 0 0"/>
+    <axis xyz="0 1 0"/>
+    <origin rpy="0 0 0" xyz="0 0 0"/>
     <parent link="fl_wheel_link"/>
     <child link="fl_wheel"/>
   </joint>
   <link name="fl_wheel">
-    <visual>
-      <orgin rpy="0 0 0" xyz="-0.7 0.8 0"/>
-      <geometry>
-        <cylinder radius="0.4" length="0.2"/>
+    <inertial>
+        <mass value="1e-4"/>
+      <origin  xyz="0 0 0" rpy="1.5708 0 0" />
+        <inertia
+          ixx="0.1" ixy="0.0" ixz="0.0"
+          iyy="0.1" iyz="0.0"
+          izz="0.1"
+        />
+      </inertial>
+    <collision>
+        <origin  xyz="0 0 0" rpy="1.5708 0 0" />
+        <geometry>
+          <cylinder radius="0.08" length="0.04"/>
+        </geometry>
+      </collision>
+    <visual>
+      <origin  xyz="0 0 0" rpy="1.5708 0 0" />
+      <geometry>
+        <cylinder radius="0.08" length="0.04"/>
       </geometry>
       <material name="black"/>
@@ -47,5 +164,5 @@
     <axis xyz="0 0 1"/>
     <limit effort="1000.0" lower="-0.4" upper="0.4" velocity="0.5"/>
-    <origin rpy="0 0 0" xyz="0.5 0.8 0"/>
+    <origin rpy="0 0 0" xyz="0.2 -0.25 0"/>
     <parent link="base"/>
     <child link="fr_wheel_link"/>
@@ -53,5 +170,5 @@
   <link name="fr_wheel_link">
     <visual>
-      <orgin rpy="0 0 0" xyz="0.7 0.8 0"/>
+      <origin rpy="0 0 0" xyz="0.7 0.8 0"/>
       <geometry>
         <box size="0 0 0"/>
@@ -61,5 +178,5 @@
   <joint name="fr_wheel_joint" type="continuous">
     <axis xyz="0 0 1"/>
-    <origin rpy="0 1.57 0" xyz="0.2 0 0"/>
+    <origin rpy="0 0 0" xyz="0 0 0"/>
     <parent link="fr_wheel_link"/>
     <child link="fr_wheel"/>
@@ -67,7 +184,7 @@
   <link name="fr_wheel">
     <visual>
-      <orgin rpy="0 0 0" xyz="0.7 0.8 0"/>
-      <geometry>
-        <cylinder radius="0.4" length="0.2"/>
+      <origin rpy="1.5707 0 0" xyz="0.7 0.8 0"/>
+      <geometry>
+        <cylinder radius="0.08" length="0.04"/>
       </geometry>
       <material name="black"/>
@@ -76,6 +193,6 @@
   <!--Rear left wheel-->
   <joint name="rl_wheel_joint" type="continuous">
-    <axis xyz="0 0 1"/>
-    <origin rpy="0 1.57 0" xyz="-0.7 -0.8 0"/>
+    <axis xyz="0 1 0"/>
+    <origin rpy="0 0 0" xyz="-0.2 0.25 0"/>
     <parent link="base"/>
     <child link="rl_wheel"/>
@@ -83,7 +200,7 @@
   <link name="rl_wheel">
     <visual>
-      <orgin rpy="0 0 0" xyz="-0.7 -0.8 0"/>
-      <geometry>
-        <cylinder radius="0.4" length="0.2"/>
+    <origin rpy="1.5708 0 0" xyz="0 0 0"/>
+      <geometry>
+        <cylinder radius="0.08" length="0.04"/>
       </geometry>
       <material name="black"/>
@@ -92,6 +209,6 @@
   <!--Rear right wheel-->
   <joint name="rr_wheel_joint" type="continuous">
-    <axis xyz="0 0 1"/>
-    <origin rpy="0 1.57 0" xyz="0.7 -0.8 0"/>
+    <axis xyz="0 1 0"/>
+    <origin rpy="1.5708 0 0" xyz="-0.2 -0.25 0"/>
     <parent link="base"/>
     <child link="rr_wheel"/>
@@ -99,7 +216,7 @@
   <link name="rr_wheel">
     <visual>
-      <orgin rpy="0 0 0" xyz="0.7 -0.8 0"/>
-      <geometry>
-        <cylinder radius="0.4" length="0.2"/>
+      <origin rpy="0 0 0" xyz="0 0 0"/>
+      <geometry>
+        <cylinder radius="0.08" length="0.04"/>
       </geometry>
       <material name="black"/>

Commit message: Añadido sensor

File: urdf/jetracer.xacro (robot description, xacro)
@@ -8,11 +8,17 @@
   </material>
   <joint name="camera_joint" type="fixed">
-      <origin xyz="0.17 0 0.1" rpy="0 0 0" />
+      <origin xyz="0.20 -0.10 0.1" rpy="0 0 0" />
       <parent link="base"/>
       <child link="camera" />
       <axis xyz="0 1 0"/>
   </joint>
-  <!-- CAMARA -->
-  <link name="camera">
+<joint name="sensor_joint" type="fixed">
+      <origin xyz="0.20 0.10 0.1" rpy="0 0 0" />
+      <parent link="base"/>
+      <child link="sensor" />
+      <axis xyz="0 1 0"/>
+  </joint>
+  <!--SENSOR-->
+<link name="sensor">
     <inertial>
       <mass value="0.1"/>
@@ -38,7 +44,32 @@
     </visual>
   </link>
+  <!-- CAMARA -->
+  <link name="camera">
+    <inertial>
+      <mass value="0.1"/>
+      <origin xyz="0 0 0" rpy="0 0 0"/>
+      <inertia
+        ixx="1e-6" ixy="0.0" ixz="0.0"
+        iyy="1e-6" iyz="0.0"
+        izz="1e-6"
+      />
+    </inertial>
+    <collision>
+      <origin xyz="0 0 0" rpy="0 0 0"/>
+      <geometry>
+        <box size="0.05 0.05 0.05"/>
+      </geometry>
+    </collision>
+    <visual>
+      <origin xyz="0 0 0" rpy="0 0 0"/>
+      <geometry>
+        <box size="0.05 0.05 0.05"/>
+      </geometry>
+      <material name="blue"/>
+    </visual>
+  </link>
   <!--LASER-->
     <joint name="hokuyo_joint" type="fixed">
-      <origin xyz="0.10 -0.03 0.15" rpy="0 0 0" />
+      <origin xyz="0.10 0 0.15" rpy="0 0 0" />
       <parent link="base"/>
       <child link="hokuyo" />
@@ -78,5 +109,5 @@
     <pose>0 0 0 0 0 0</pose>
     <inertial>
-      <mass value="25.0"/>
+      <mass value="0.2"/>
       <origin xyz="0 0 0.05" rpy=" 0 0 0"/>
       <inertia
@@ -162,5 +193,5 @@
   <!--Front right wheel-->
   <joint name="fr_holder_joint" type="revolute">
-    <axis xyz="0 0 1"/>
+    <axis xyz="1 0 0"/>
     <limit effort="1000.0" lower="-0.4" upper="0.4" velocity="0.5"/>
     <origin rpy="0 0 0" xyz="0.2 -0.25 0"/>
@@ -169,7 +200,22 @@
   </joint>
   <link name="fr_wheel_link">
-    <visual>
-      <origin rpy="0 0 0" xyz="0.7 0.8 0"/>
-      <geometry>
+    <inertial>
+      <mass value="1e-4"/>
+      <origin rpy="0 0 0" xyz="0.7 0.8 0"/>
+      <inertia
+        ixx="0.1" ixy="0.0" ixz="0.0"
+        iyy="0.1" iyz="0.0"
+        izz="0.1"
+      />
+    </inertial>
+    <collision>
+     <origin rpy="0 0 0" xyz="0.7 0.8 0"/>
+      <geometry>
+        <box size="0 0 0"/>
+      </geometry>
+    </collision>
+    <visual>
+      <origin rpy="0 0 0" xyz="0.7 0.8 0"/>
+     <geometry>
         <box size="0 0 0"/>
       </geometry>
@@ -177,5 +223,5 @@
   </link>
   <joint name="fr_wheel_joint" type="continuous">
-    <axis xyz="0 0 1"/>
+    <axis xyz="0 1 0"/>
     <origin rpy="0 0 0" xyz="0 0 0"/>
     <parent link="fr_wheel_link"/>
@@ -183,6 +229,21 @@
   </joint>
   <link name="fr_wheel">
-    <visual>
-      <origin rpy="1.5707 0 0" xyz="0.7 0.8 0"/>
+    <inertial>
+        <mass value="1e-4"/>
+      <origin  xyz="0 0 0" rpy="1.5708 0 0" />
+        <inertia
+          ixx="0.1" ixy="0.0" ixz="0.0"
+          iyy="0.1" iyz="0.0"
+          izz="0.1"
+        />
+      </inertial>
+    <collision>
+        <origin  xyz="0 0 0" rpy="1.5708 0 0" />
+        <geometry>
+          <cylinder radius="0.08" length="0.04"/>
+        </geometry>
+      </collision>
+    <visual>
+      <origin  xyz="0 0 0" rpy="1.5708 0 0" />
       <geometry>
         <cylinder radius="0.08" length="0.04"/>
